File: RC Transmitter/PCB/TransmitterV2/TransmitterV2.kicad_pcb (KiCad board)
At the start: 2 copper layers, 35.6 x 99.8 mm, 78 parts, among them J1 Conn_01x06, J2 USB_B_Micro, J3 Conn_01x03, J4 Conn_01x03, J5 Conn_01x08, J6 Conn_01x06, J7 Conn_01x02, SW1 SW_Push_45deg, SW2 SW_Push_45deg, SW3 SW_Push_45deg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

Commit message: add 3D designs
Parts:
- moved R14 7.82 mm to (127.6, 99.9)
Connections:
- J3 pad 2: D8 -> unconnected-(J3-Pad2)
- J4 pad 2: D7 -> unconnected-(J4-Pad2)
Routing:
- net D8: track 29.1 -> 21.2 mm
- net D7: track 60.5 -> 64.6 mm
- net GND: vias 86 -> 83
Changed lines of the file:
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@@
   (net 68 "unconnected-(U4-Pad15)")
   (net 69 "unconnected-(U6-Pad6)")
+  (net 70 "unconnected-(J3-Pad2)")
+  (net 71 "unconnected-(J4-Pad2)")
   (footprint "Capacitor_SMD:C_0805_2012Metric_Pad1.18x1.45mm_HandSolder" (layer "F.Cu")
     (at 131.318 39.6455 90)
@@
       (net 3 "+3V3") (pinfunction "Pin_1") (pintype "passive"))
     (pad "2" smd roundrect (at 0 9.144) (size 6 3) (layers "F.Cu" "F.Paste" "F.Mask") (roundrect_rratio 0.25)
-      (net 31 "D7") (pinfunction "Pin_2") (pintype "passive"))
+      (net 71 "unconnected-(J4-Pad2)") (pinfunction "Pin_2") (pintype "passive"))
     (pad "3" smd roundrect (at 0 16.256) (size 6 3) (layers "F.Cu" "F.Paste" "F.Mask") (roundrect_rratio 0.25)
       (net 31 "D7") (pinfunction "Pin_3") (pintype "passive"))
@@
       (net 3 "+3V3") (pinfunction "Pin_1") (pintype "passive"))
     (pad "2" smd roundrect (at 0 9.144 180) (size 6 3) (layers "F.Cu" "F.Paste" "F.Mask") (roundrect_rratio 0.25)
-      (net 30 "D8") (pinfunction "Pin_2") (pintype "passive"))
+      (net 70 "unconnected-(J3-Pad2)") (pinfunction "Pin_2") (pintype "passive"))
     (pad "3" smd roundrect (at 0 16.256 180) (size 6 3) (layers "F.Cu" "F.Paste" "F.Mask") (roundrect_rratio 0.25)
       (net 30 "D8") (pinfunction "Pin_3") (pintype "passive"))
@@
   )
   (footprint "Resistor_SMD:R_0805_2012Metric" (layer "F.Cu")
-    (at 127.762 107.696 180)
+    (at 127.6115 99.8728 180)
     (descr "Resistor SMD 0805 (2012 Metric), square (rectangular) end terminal, IPC_7351 nominal, (Body size source: IPC-SM-782 page 72, https://www.pcb-3d.com/wordpress/wp-content/uploads/ipc-sm-782a_amendment_1_and_2.pdf), generated with kicad-footprint-generator")
     (tags "resistor")
@@
   (via (at 133.35 88.9) (size 0.8) (drill 0.4) (layers "F.Cu" "B.Cu") (free) (net 1))
   (via (at 147.32 93.218) (size 0.8) (drill 0.4) (layers "F.Cu" "B.Cu") (free) (net 1))
-  (via (at 129.54 100.965) (size 0.8) (drill 0.4) (layers "F.Cu" "B.Cu") (free) (net 1))
   (via (at 151.892 102.108) (size 0.8) (drill 0.4) (layers "F.Cu" "B.Cu") (free) (net 1))
   (via (at 149.352 85.344) (size 0.8) (drill 0.4) (layers "F.Cu" "B.Cu") (free) (net 1))
@@
   (via (at 143.764 110.236) (size 0.8) (drill 0.4) (layers "F.Cu" "B.Cu") (free) (net 1))
   (via (at 151.13 64.135) (size 0.8) (drill 0.4) (layers "F.Cu" "B.Cu") (net 1))
-  (via (at 129.54 99.06) (size 0.8) (drill 0.4) (layers "F.Cu" "B.Cu") (free) (net 1))
-  (via (at 127 99.695) (size 0.8) (drill 0.4) (layers "F.Cu" "B.Cu") (free) (net 1))
   (via (at 142.875 114.935) (size 0.8) (drill 0.4) (layers "F.Cu" "B.Cu") (free) (net 1))
   (via (at 128.016 43.688) (size 0.8) (drill 0.4) (layers "F.Cu" "B.Cu") (free) (net 1))
@@
   (segment (start 147.001 65.659) (end 150.495 65.659) (width 0.2) (layer "B.Cu") (net 28))
   (segment (start 150.495 65.659) (end 150.622 65.786) (width 0.2) (layer "B.Cu") (net 28))
-  (segment (start 128.6745 107.696) (end 128.6745 103.5285) (width 0.25) (layer "F.Cu") (net 30))
-  (segment (start 128.6745 103.5285) (end 128.524 103.378) (width 0.25) (layer "F.Cu") (net 30))
+  (segment (start 128.524 99.8728) (end 128.524 96.266) (width 0.25) (layer "F.Cu") (net 30))
   (segment (start 133.354299 85.094299) (end 129.781087 85.094299) (width 0.25) (layer "F.Cu") (net 30))
   (segment (start 128.524 86.351386) (end 128.524 96.266) (width 0.25) (layer "F.Cu") (net 30))
-  (segment (start 128.524 103.378) (end 128.524 96.266) (width 0.25) (layer "F.Cu") (net 30))
   (segment (start 129.781087 85.094299) (end 128.524 86.351386) (width 0.25) (layer "F.Cu") (net 30))
   (via (at 133.354299 85.094299) (size 0.8) (drill 0.4) (layers "F.Cu" "B.Cu") (net 30))
   (segment (start 134.004 82.99) (end 134.004 84.444598) (width 0.25) (layer "B.Cu") (net 30))
   (segment (start 134.004 84.444598) (end 133.354299 85.094299) (width 0.25) (layer "B.Cu") (net 30))
-  (segment (start 128.571 122.682) (end 128.571 127.207) (width 0.25) (layer "F.Cu") (net 31))
-  (segment (start 128.524 127.254) (end 128.524 134.366) (width 0.25) (layer "F.Cu") (net 31))
+  (segment (start 129.8956 122.682) (end 132.5372 125.3236) (width 0.25) (layer "F.Cu") (net 31))
+  (segment (start 132.5372 125.3236) (end 132.5372 130.3528) (width 0.25) (layer "F.Cu") (net 31))
+  (segment (start 132.5372 130.3528) (end 128.524 134.366) (width 0.25) (layer "F.Cu") (net 31))
   (segment (start 128.571 122.682) (end 125.19948 119.31048) (width 0.25) (layer "F.Cu") (net 31))
   (segment (start 128.07448 92.025134) (end 128.07448 86.165189) (width 0.25) (layer "F.Cu") (net 31))
+  (segment (start 128.571 122.682) (end 129.8956 122.682) (width 0.25) (layer "F.Cu") (net 31))
   (segment (start 129.869881 84.369788) (end 133.691729 84.369788) (width 0.25) (layer "F.Cu") (net 31))
   (segment (start 133.691729 84.369788) (end 134.461989 85.140048) (width 0.25) (layer "F.Cu") (net 31))
   (segment (start 125.19948 119.31048) (end 125.19948 94.900134) (width 0.25) (layer "F.Cu") (net 31))
   (segment (start 128.07448 86.165189) (end 129.869881 84.369788) (width 0.25) (layer "F.Cu") (net 31))
-  (segment (start 128.571 127.207) (end 128.524 127.254) (width 0.25) (layer "F.Cu") (net 31))
   (segment (start 125.19948 94.900134) (end 128.07448 92.025134) (width 0.25) (layer "F.Cu") (net 31))
   (via (at 134.461989 85.140048) (size 0.8) (drill 0.4) (layers "F.Cu" "B.Cu") (net 31))
@@
   (segment (start 147.828 115.062) (end 147.828 110.236) (width 0.25) (layer "B.Cu") (net 60))
   (segment (start 146.304 92.202) (end 146.304 108.712) (width 0.25) (layer "B.Cu") (net 60))
+  (segment (start 128.6745 103.5285) (end 128.524 103.378) (width 0.25) (layer "F.Cu") (net 70))
+  (segment (start 128.571 127.207) (end 128.524 127.254) (width 0.25) (layer "F.Cu") (net 71))
   (zone (net 1) (net_name "GND") (layer "F.Cu") (hatch edge 0.508)
     (connect_pads (clearance 0.3))
