File: RC Transmitter/PCB/TransmitterV2/TransmitterV2.kicad_sch (KiCad schematic)
At the start: 78 parts, among them J1 Conn_01x06, J2 USB_B_Micro, J3 Conn_01x03, J4 Conn_01x03, J5 Conn_01x08, J6 Conn_01x06, J7 Conn_01x02, SW1 SW_Push_45deg, SW2 SW_Push_45deg, SW3 SW_Push_45deg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

Commit message: add 3D designs
Connections:
- net D7: no longer J4.2 (Pin_2)
- net D8: no longer J3.2 (Pin_2)
Changed lines of the file:
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@@
 (kicad_sch (version 20211123) (generator eeschema)
   (paper "A4")
-  (junction (at 111.76 24.13) (diameter 0) (color 0 0 0 0)
-  )
   (junction (at 48.26 105.41) (diameter 0) (color 0 0 0 0)
   )
@@
   )
   (junction (at 132.08 87.63) (diameter 0) (color 0 0 0 0)
-  )
-  (junction (at 111.76 34.29) (diameter 0) (color 0 0 0 0)
   )
   (junction (at 26.67 121.92) (diameter 0) (color 0 0 0 0)
@@
     (stroke (width 0) (type default) (color 0 0 0 0))
   )
-  (wire (pts (xy 114.3 33.02) (xy 111.76 33.02))
-    (stroke (width 0) (type default) (color 0 0 0 0))
-  )
   (wire (pts (xy 43.18 111.76) (xy 43.18 113.03))
     (stroke (width 0) (type default) (color 0 0 0 0))
@@
     (stroke (width 0) (type default) (color 0 0 0 0))
   )
-  (wire (pts (xy 111.76 33.02) (xy 111.76 34.29))
-    (stroke (width 0) (type default) (color 0 0 0 0))
-  )
   (wire (pts (xy 40.64 71.12) (xy 40.64 77.47))
     (stroke (width 0) (type default) (color 0 0 0 0))
@@
     (stroke (width 0) (type default) (color 0 0 0 0))
   )
-  (wire (pts (xy 111.76 22.86) (xy 111.76 24.13))
-    (stroke (width 0) (type default) (color 0 0 0 0))
-  )
   (wire (pts (xy 85.09 72.39) (xy 87.63 72.39))
     (stroke (width 0) (type default) (color 0 0 0 0))
@@
     (stroke (width 0) (type default) (color 0 0 0 0))
   )
-  (wire (pts (xy 114.3 22.86) (xy 111.76 22.86))
-    (stroke (width 0) (type default) (color 0 0 0 0))
-  )
